File: STM32WL55JC_pcb_design/STM32WL55JC_pcb_design.sch (KiCad schematic (older format))
At the start: 27 parts

Commit message: First pcb commit
Parts:
- U?: symbol MCU_ST_STM3255JCI7:STM32WL55JCI7 -> STM32WL55JC_pcb_design-rescue:STM32WL55JCI7-MCU_ST_STM3255JCI7
Changed lines of the file:
@@
 	2950 2250 3100 2250
 $Comp
-L MCU_ST_STM3255JCI7:STM32WL55JCI7 U?
+L STM32WL55JC_pcb_design-rescue:STM32WL55JCI7-MCU_ST_STM3255JCI7 U?
 U 1 1 61223ADA
 P 5350 1900
