File: STM32WL55JC_pcb_design/STM32WL55JC_pcb_design.sch (KiCad schematic (older format))
At the start: 36 parts, among them IC1 STM32F051R8T6, J1 Conn_01x03, J10 Conn_01x08_Male, J11 Conn_02x02_Odd_Even, J2 Conn_01x03, J22 Conn_01x19_Male, J3 Conn_01x03, J4 Conn_01x09, J5 Conn_01x09, J6 Conn_01x03, J7 Conn_01x09, J8 Conn_01x09, J9 Conn_02x10_Odd_Even, Y1 32MHz, Y2 32.768kHz

Commit message: Final push
Other:
- moved on the sheet: TP1, TP2
Changed lines of the file:
@@
 Text Notes 9550 8200 0    50   ~ 0
 External clocks
-$Comp
-L Device:Crystal_GND24 Y1
-U 1 1 6176899B
-P 10400 6450
-F 0 "Y1" H 10350 6850 50  0000 L CNN
-F 1 "32MHz" H 10300 6750 50  0000 L CNN
-F 2 "NX2016SA32MEXS00ACS06465:NX2016SA32MEXS00ACS06465" H 10400 6450 50  0001 C CNN
-F 3 "~" H 10400 6450 50  0001 C CNN
-	1    10400 6450
-	1    0    0    -1
-$EndComp
 Wire Wire Line
 	10400 6250 10600 6250
@@
 P 6250 3950
 F 0 "IC1" H 8394 3246 50  0000 L CNN
-F 1 "STM32F051R8T6" H 8394 3155 50  0000 L CNN
+F 1 "STM32F051R8T6" H 7000 3150 50  0000 L CNN
 F 2 "STM32F051R8T6:QFP50P1200X1200X160-64N" H 8200 4450 50  0001 L CNN
 F 3 "http://www.st.com/web/en/resource/technical/document/datasheet/DM00039193.pdf" H 8200 4350 50  0001 L CNN
@@
 Text GLabel 10700 2300 2    50   Input ~ 0
 EXP_P5
-Text GLabel 6900 7700 3    50   Input ~ 0
+Text GLabel 6750 7750 3    50   Input ~ 0
 VDD
 $Comp
 L power:GNDREF #PWR0101
 U 1 1 61855E4F
-P 7400 7700
-F 0 "#PWR0101" H 7400 7450 50  0001 C CNN
-F 1 "GNDREF" H 7405 7527 50  0000 C CNN
-F 2 "" H 7400 7700 50  0001 C CNN
-F 3 "" H 7400 7700 50  0001 C CNN
-	1    7400 7700
+P 7250 7750
+F 0 "#PWR0101" H 7250 7500 50  0001 C CNN
+F 1 "GNDREF" H 7255 7577 50  0000 C CNN
+F 2 "" H 7250 7750 50  0001 C CNN
+F 3 "" H 7250 7750 50  0001 C CNN
+	1    7250 7750
 	1    0    0    -1
 $EndComp
@@
 L Connector:TestPoint TP1
 U 1 1 618577EB
-P 6900 7700
-F 0 "TP1" H 6958 7818 50  0000 L CNN
-F 1 "Micro_VDD" H 6958 7727 50  0000 L CNN
-F 2 "TestPoint:TestPoint_Pad_D4.0mm" H 7100 7700 50  0001 C CNN
-F 3 "~" H 7100 7700 50  0001 C CNN
-	1    6900 7700
+P 6750 7750
+F 0 "TP1" H 6808 7868 50  0000 L CNN
+F 1 "Micro_VDD" H 6808 7777 50  0000 L CNN
+F 2 "TestPoint:TestPoint_Pad_D4.0mm" H 6950 7750 50  0001 C CNN
+F 3 "~" H 6950 7750 50  0001 C CNN
+	1    6750 7750
 	1    0    0    -1
 $EndComp
@@
 L Connector:TestPoint TP2
 U 1 1 61858267
-P 7400 7700
-F 0 "TP2" H 7458 7818 50  0000 L CNN
-F 1 "Micro_GND" H 7458 7727 50  0000 L CNN
-F 2 "TestPoint:TestPoint_Pad_D4.0mm" H 7600 7700 50  0001 C CNN
-F 3 "~" H 7600 7700 50  0001 C CNN
-	1    7400 7700
-	1    0    0    -1
-$EndComp
+P 7250 7750
+F 0 "TP2" H 7308 7868 50  0000 L CNN
+F 1 "Micro_GND" H 7308 7777 50  0000 L CNN
+F 2 "TestPoint:TestPoint_Pad_D4.0mm" H 7450 7750 50  0001 C CNN
+F 3 "~" H 7450 7750 50  0001 C CNN
+	1    7250 7750
+	1    0    0    -1
+$EndComp
+$Comp
+L Device:Crystal_GND24 Y1
+U 1 1 6176899B
+P 10400 6450
+F 0 "Y1" H 10350 6850 50  0000 L CNN
+F 1 "32MHz" H 10300 6750 50  0000 L CNN
+F 2 "NX2016SA32MEXS00ACS06465:NX2016SA32MEXS00ACS06465" H 10400 6450 50  0001 C CNN
+F 3 "~" H 10400 6450 50  0001 C CNN
+	1    10400 6450
+	1    0    0    -1
+$EndComp
