File: STM32WL55JC_pcb_design/ExpanderPlusEncoders.sch (KiCad schematic (older format))
At the start: 10 parts, among them IC2 CY8C9540A-24PVXIT, J12 Conn_01x10, J13 Conn_01x10, J14 Conn_01x10, J15 Conn_01x10, SW2 SW_MEC_5E

Commit message: Finish pcb routing
Parts:
- added C49: 100nF, Capacitor_SMD:C_0805_2012Metric, symbol Device:C_Small
Connections:
- net EXP_GND: now also C49.2
- net EXP_VDD: now also C49.1
Changed lines of the file:
@@
 Text HLabel 5700 4700 0    50   Input ~ 0
 EXP_GND
-Text HLabel 8500 2400 2    50   Input ~ 0
+Text HLabel 9100 2400 2    50   Input ~ 0
 EXP_VDD
 $Comp
@@
 Wire Wire Line
 	9550 3700 9750 3700
+$Comp
+L Device:C_Small C49
+U 1 1 6192549B
+P 9000 2500
+F 0 "C49" H 9092 2546 50  0000 L CNN
+F 1 "100nF" H 9092 2455 50  0000 L CNN
+F 2 "Capacitor_SMD:C_0805_2012Metric" H 9000 2500 50  0001 C CNN
+F 3 "~" H 9000 2500 50  0001 C CNN
+	1    9000 2500
+	1    0    0    -1
+$EndComp
+Wire Wire Line
+	8500 2400 9000 2400
+Wire Wire Line
+	9000 2400 9100 2400
+Connection ~ 9000 2400
+Text HLabel 9100 2600 2    50   Input ~ 0
+EXP_GND
+Wire Wire Line
+	9000 2600 9100 2600
 $EndSCHEMATC
