File: STM32WL55JC_pcb_design/LoRa.sch (KiCad schematic (older format))
At the start: 55 parts, among them IC2 CG2409M2, IC3 SX1276IMLTRT, IC4 CG2409M2, J16 Conn_Coaxial, J17 Conn_Coaxial, Y3 32MHz

Commit message: Finish silk screen
Parts:
- added TP3: LoRa_VDD, TestPoint:TestPoint_Pad_D4.0mm, symbol Connector:TestPoint
- added TP4: LoRa_GND, TestPoint:TestPoint_Pad_D4.0mm, symbol Connector:TestPoint
Connections:
- net GNDREF: now also TP4.1
- new net VDD: TP3.1
Changed lines of the file:
@@
 	1    0    0    -1
 $EndComp
-Connection ~ 2350 1450
 Wire Wire Line
 	2150 1150 3050 1150
@@
 	0    1    1    0
 $EndComp
+$Comp
+L Connector:TestPoint TP3
+U 1 1 6183469E
+P 4450 750
+F 0 "TP3" H 4508 868 50  0000 L CNN
+F 1 "LoRa_VDD" H 4508 777 50  0000 L CNN
+F 2 "TestPoint:TestPoint_Pad_D4.0mm" H 4650 750 50  0001 C CNN
+F 3 "~" H 4650 750 50  0001 C CNN
+	1    4450 750
+	1    0    0    -1
+$EndComp
+$Comp
+L Connector:TestPoint TP4
+U 1 1 61849598
+P 4900 750
+F 0 "TP4" H 4958 868 50  0000 L CNN
+F 1 "LoRa_GND" H 4958 777 50  0000 L CNN
+F 2 "TestPoint:TestPoint_Pad_D4.0mm" H 5100 750 50  0001 C CNN
+F 3 "~" H 5100 750 50  0001 C CNN
+	1    4900 750
+	1    0    0    -1
+$EndComp
+$Comp
+L power:GNDREF #PWR0102
+U 1 1 61875071
+P 4900 750
+F 0 "#PWR0102" H 4900 500 50  0001 C CNN
+F 1 "GNDREF" H 4905 577 50  0000 C CNN
+F 2 "" H 4900 750 50  0001 C CNN
+F 3 "" H 4900 750 50  0001 C CNN
+	1    4900 750
+	1    0    0    -1
+$EndComp
+Connection ~ 2350 1450
+Text GLabel 4450 750  3    50   Input ~ 0
+VDD
 $EndSCHEMATC
